File: hardware/xmas_v4/xmas_v4.sch (EAGLE design)
At the start: 35 parts, among them J1 AVR_SPI_PROG_3X2TESTPOINTS, Q1 2N3904, Q2 SI2305, Q3 SI2305, U1 ATTINY85-20SU, U2 NCP1402SN50T1G

Commit message: Added schematic
Parts:
- renumbered L10 to L1, L11 to L0, L8 to L3, L9 to L2
Connections:
- net N$11: now also L4.DIN; no longer L7.DIN
- net N$12: now also L6.DOUT, L7.DIN; no longer L4.DIN, L5.DOUT
- net N$13: now also L5.DOUT, L6.DIN; no longer L5.DIN, L6.DOUT
- net N$14: now also L4.DOUT, L5.DIN; no longer L6.DIN, L7.DOUT
Other:
- moved on the sheet: 47UH, C1, C2, D1, D2, D3, J1, J3, J4, L4, L5, L6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
